File: KiCAD/Egg/Egg.kicad_pcb (KiCad board)
At the start: 2 copper layers, 11 parts, among them J1 Conn_01x05_NFC, J2 Conn_01x03_Female_VibrationMo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

Commit message: finish PCB
Parts:
- BT1, J1: moved to B.Cu
- moved J2 68.3 mm to (88.8, 96.3)
- moved J1 65.2 mm to (100.2, 109.0), turned to 180 degrees
- moved D2 60.0 mm to (80.6, 98.7)
- moved D3 54.4 mm to (85.6, 109.7)
- moved D4 45.7 mm to (115.3, 109.7)
- moved D1 42.2 mm to (85.6, 87.0)
- moved BT1 34.1 mm to (100.2, 81.3), turned to 270 degrees
- moved H1 33.1 mm to (112.6, 93.6)
- moved D5 27.1 mm to (120.4, 98.6)
- moved D6 8.85 mm to (115.1, 87.0)
- moved A1 1.09 mm to (92.5, 80.9)
Connections:
- BT1 pad 1: +7.5V -> +5V
- BT1 pad 2: GNDPWR -> GND
Routing:
- net +5V: track 0.00 -> 135.6 mm
- net GND: track 0.00 -> 115.6 mm
- net Net-(D3-Pad2): track 0.00 -> 47.9 mm
- net /RGBW: track 0.00 -> 22.2 mm
- net /VibrationMotor: track 0.00 -> 21.9 mm
- net Net-(D4-Pad2): track 0.00 -> 20.6 mm
- net /SCL: track 0.00 -> 18.4 mm
- net Net-(D5-Pad2): track 0.00 -> 16.5 mm
- net /SDA: track 0.00 -> 15.3 mm
- net Net-(D2-Pad2): track 0.00 -> 13.1 mm
- net /SCK: track 0.00 -> 9.04 mm
- net Net-(D1-Pad2): track 0.00 -> 8.51 mm
- net Net-(D6-Pad2): track 0.00 -> 5.02 mm
Other:
- board outline added: 50 x 50 mm

Commit message: NFC ini
Parts:
- removed H1: MountingHole_Pad, Connector_PinHeader_1.00mm:PinHeader_1x01_P1.00mm_Vertical
- BT1: footprint Connector_AMASS:AMASS_XT30U-F_1x02_P5.0mm_Vertical -> Connector_JST:JST_PH_B2B-PH-K_1x02_P2.00mm_Vertical
- J1: value Conn_01x05_NFC -> Conn_01x04_NFC; footprint Connector_JST:JST_GH_BM05B-GHS-TBT_1x05-1MP_P1.25mm_Vertical -> Connector_JST:JST_GH_BM04B-GHS-TBT_1x04-1MP_P1.25mm_Vertical
Connections:
- A1 pad 1: /VibrationMotor -> (no net)
- A1 pad 10: /NFC1 -> (no net)
- A1 pad 11: /NFC2 -> (no net)
- A1 pad 12: Net-(A1-Pad12) -> (no net)
- A1 pad 13: Net-(A1-Pad13) -> (no net)
- A1 pad 14: Net-(A1-Pad14) -> (no net)
- A1 pad 15: Net-(A1-Pad15) -> (no net)
- A1 pad 16: /SCK -> (no net)
- A1 pad 17: Net-(A1-Pad17) -> (no net)
- A1 pad 18: Net-(A1-Pad18) -> (no net)
- A1 pad 19: Net-(A1-Pad19) -> (no net)
- A1 pad 2: Net-(A1-Pad2) -> (no net)
- A1 pad 20: Net-(A1-Pad20) -> (no net)
- A1 pad 21: Net-(A1-Pad21) -> (no net)
- A1 pad 22: Net-(A1-Pad22) -> (no net)
- A1 pad 25: Net-(A1-Pad25) -> (no net)
- A1 pad 26: Net-(A1-Pad26) -> (no net)
- A1 pad 28: Net-(A1-Pad28) -> (no net)
- A1 pad 3: Net-(A1-Pad3) -> (no net)
- A1 pad 30: Net-(A1-Pad30) -> (no net)
- A1 pad 5: Net-(A1-Pad5) -> /VibrationMotor
- A1 pad 6: Net-(A1-Pad6) -> (no net)
- A1 pad 7: Net-(A1-Pad7) -> (no net)
- A1 pad 8: Net-(A1-Pad8) -> (no net)
- D6 pad 2: Net-(D6-Pad2) -> (no net)
- J1 pad 2: /SCK -> /SDA
- J1 pad 3: /SDA -> /SCL
- J1 pad 4: /SCL -> GND
Routing:
- net /VibrationMotor: track 21.9 -> 9.27 mm
- net /SCK: track 9.04 -> 0.00 mm
- net GND: track 115.6 -> 123.8 mm
- net Net-(D6-Pad2): track 5.02 -> 0.00 mm
- net +5V: track 135.6 -> 136.4 mm
