File: KiCAD/Egg/Egg.sch (KiCad schematic (older format))
At the start: 1 part

Commit message: INI
Parts:
- added BT?: Battery_Cell, Connector_AMASS:AMASS_XT30U-F_1x02_P5.0mm_Vertical, symbol Device:Battery_Cell
- added D? (x6): WS2812B, LED_SMD:LED_WS2812B_PLCC4_5.0x5.0mm_P3.2mm, symbol LED:WS2812B
- added H?: MountingHole_Pad, Connector_PinHeader_1.00mm:PinHeader_1x01_P1.00mm_Vertical, symbol Mechanical:MountingHole_Pad
Connections:
- net NFC1: now reaches A?.10 (D7)
- net NFC2: now reaches A?.11 (D8)
- net RGBW: now reaches A?.9 (D6)
- net RGBW: now also D?.4 (DIN)
- new net: D?.2 (DOUT), D?.4 (DIN) (x5)
- new net: D?.2 (DOUT), H?.1
- new net +5V: D?.1 (VDD), D?.1 (VDD), D?.1 (VDD), D?.1 (VDD), D?.1 (VDD), D?.1 (VDD)
- new net +7.5V: BT?.1 (+)
- new net GND: D?.3 (VSS), D?.3 (VSS), D?.3 (VSS), D?.3 (VSS), D?.3 (VSS), D?.3 (VSS)
- new net GNDPWR: BT?.2 (-)
Changed lines of the file:
@@
 	1    0    0    -1
 $EndComp
+$Comp
+L LED:WS2812B D?
+U 1 1 5F6043E7
+P 1100 1100
+F 0 "D?" H 1444 1146 50  0000 L CNN
+F 1 "WS2812B" H 1444 1055 50  0000 L CNN
+F 2 "LED_SMD:LED_WS2812B_PLCC4_5.0x5.0mm_P3.2mm" H 1150 800 50  0001 L TNN
+F 3 "https://cdn-shop.adafruit.com/datasheets/WS2812B.pdf" H 1200 725 50  0001 L TNN
+	1    1100 1100
+	1    0    0    -1
+$EndComp
+$Comp
+L LED:WS2812B D?
+U 1 1 5F606A1F
+P 2100 1100
+F 0 "D?" H 2444 1146 50  0000 L CNN
+F 1 "WS2812B" H 2444 1055 50  0000 L CNN
+F 2 "LED_SMD:LED_WS2812B_PLCC4_5.0x5.0mm_P3.2mm" H 2150 800 50  0001 L TNN
+F 3 "https://cdn-shop.adafruit.com/datasheets/WS2812B.pdf" H 2200 725 50  0001 L TNN
+	1    2100 1100
+	1    0    0    -1
+$EndComp
+$Comp
+L LED:WS2812B D?
+U 1 1 5F608368
+P 3100 1100
+F 0 "D?" H 3444 1146 50  0000 L CNN
+F 1 "WS2812B" H 3444 1055 50  0000 L CNN
+F 2 "LED_SMD:LED_WS2812B_PLCC4_5.0x5.0mm_P3.2mm" H 3150 800 50  0001 L TNN
+F 3 "https://cdn-shop.adafruit.com/datasheets/WS2812B.pdf" H 3200 725 50  0001 L TNN
+	1    3100 1100
+	1    0    0    -1
+$EndComp
+$Comp
+L LED:WS2812B D?
+U 1 1 5F60C729
+P 4100 1100
+F 0 "D?" H 4444 1146 50  0000 L CNN
+F 1 "WS2812B" H 4444 1055 50  0000 L CNN
+F 2 "LED_SMD:LED_WS2812B_PLCC4_5.0x5.0mm_P3.2mm" H 4150 800 50  0001 L TNN
+F 3 "https://cdn-shop.adafruit.com/datasheets/WS2812B.pdf" H 4200 725 50  0001 L TNN
+	1    4100 1100
+	1    0    0    -1
+$EndComp
+$Comp
+L LED:WS2812B D?
+U 1 1 5F60D2EA
+P 5100 1100
+F 0 "D?" H 5444 1146 50  0000 L CNN
+F 1 "WS2812B" H 5444 1055 50  0000 L CNN
+F 2 "LED_SMD:LED_WS2812B_PLCC4_5.0x5.0mm_P3.2mm" H 5150 800 50  0001 L TNN
+F 3 "https://cdn-shop.adafruit.com/datasheets/WS2812B.pdf" H 5200 725 50  0001 L TNN
+	1    5100 1100
+	1    0    0    -1
+$EndComp
+$Comp
+L LED:WS2812B D?
+U 1 1 5F60E008
+P 6100 1100
+F 0 "D?" H 6444 1146 50  0000 L CNN
+F 1 "WS2812B" H 6444 1055 50  0000 L CNN
+F 2 "LED_SMD:LED_WS2812B_PLCC4_5.0x5.0mm_P3.2mm" H 6150 800 50  0001 L TNN
+F 3 "https://cdn-shop.adafruit.com/datasheets/WS2812B.pdf" H 6200 725 50  0001 L TNN
+	1    6100 1100
+	1    0    0    -1
+$EndComp
+$Comp
+L power:GND #PWR?
+U 1 1 5F623C17
+P 6100 1500
+F 0 "#PWR?" H 6100 1250 50  0001 C CNN
+F 1 "GND" H 6105 1327 50  0000 C CNN
+F 2 "" H 6100 1500 50  0001 C CNN
+F 3 "" H 6100 1500 50  0001 C CNN
+	1    6100 1500
+	1    0    0    -1
+$EndComp
+$Comp
+L power:+5V #PWR?
+U 1 1 5F6244C7
+P 6100 700
+F 0 "#PWR?" H 6100 550 50  0001 C CNN
+F 1 "+5V" H 6115 873 50  0000 C CNN
+F 2 "" H 6100 700 50  0001 C CNN
+F 3 "" H 6100 700 50  0001 C CNN
+	1    6100 700
+	1    0    0    -1
+$EndComp
+Wire Wire Line
+	1100 800  1100 750
+Wire Wire Line
+	1100 750  2100 750
+Wire Wire Line
+	6100 750  6100 700
+Wire Wire Line
+	2100 800  2100 750
+Connection ~ 2100 750
+Wire Wire Line
+	2100 750  3100 750
+Wire Wire Line
+	3100 800  3100 750
+Connection ~ 3100 750
+Wire Wire Line
+	3100 750  4100 750
+Wire Wire Line
+	4100 800  4100 750
+Connection ~ 4100 750
+Wire Wire Line
+	4100 750  5100 750
+Wire Wire Line
+	5100 800  5100 750
+Connection ~ 5100 750
+Wire Wire Line
+	5100 750  6100 750
+Wire Wire Line
+	6100 800  6100 750
+Connection ~ 6100 750
+Wire Wire Line
+	1100 1400 1100 1450
+Wire Wire Line
+	1100 1450 2100 1450
+Wire Wire Line
+	6100 1450 6100 1500
+Wire Wire Line
+	6100 1400 6100 1450
+Connection ~ 6100 1450
+Wire Wire Line
+	5100 1400 5100 1450
+Connection ~ 5100 1450
+Wire Wire Line
+	5100 1450 6100 1450
+Wire Wire Line
+	4100 1400 4100 1450
+Connection ~ 4100 1450
+Wire Wire Line
+	4100 1450 5100 1450
+Wire Wire Line
+	3100 1400 3100 1450
+Connection ~ 3100 1450
+Wire Wire Line
+	3100 1450 4100 1450
+Wire Wire Line
+	2100 1400 2100 1450
+Connection ~ 2100 1450
+Wire Wire Line
+	2100 1450 3100 1450
+Wire Wire Line
+	1400 1100 1800 1100
+Wire Wire Line
+	2400 1100 2800 1100
+Wire Wire Line
+	3400 1100 3800 1100
+Wire Wire Line
+	4400 1100 4800 1100
+Wire Wire Line
+	5400 1100 5800 1100
+Wire Wire Line
+	800  1100 600  1100
+Wire Wire Line
+	6400 1100 6800 1100
+Text Label 3050 3300 0    50   ~ 0
+RGBW
+Wire Wire Line
+	3050 3300 3250 3300
+Text Label 600  1100 0    50   ~ 0
+RGBW
+Wire Wire Line
+	3250 3400 3050 3400
+Wire Wire Line
+	3250 3500 3050 3500
+Text Label 3050 3400 0    50   ~ 0
+NFC1
+Text Label 3050 3500 0    50   ~ 0
+NFC2
+$Comp
+L Mechanical:MountingHole_Pad H?
+U 1 1 5F64094E
+P 6800 1000
+F 0 "H?" H 6900 1049 50  0000 L CNN
+F 1 "MountingHole_Pad" H 6900 958 50  0000 L CNN
+F 2 "Connector_PinHeader_1.00mm:PinHeader_1x01_P1.00mm_Vertical" H 6800 1000 50  0001 C CNN
+F 3 "~" H 6800 1000 50  0001 C CNN
+	1    6800 1000
+	1    0    0    -1
+$EndComp
+$Comp
+L Device:Battery_Cell BT?
+U 1 1 5F642495
+P 6650 2950
+F 0 "BT?" H 6768 3046 50  0000 L CNN
+F 1 "Battery_Cell" H 6768 2955 50  0000 L CNN
+F 2 "Connector_AMASS:AMASS_XT30U-F_1x02_P5.0mm_Vertical" V 6650 3010 50  0001 C CNN
+F 3 "~" V 6650 3010 50  0001 C CNN
+	1    6650 2950
+	1    0    0    -1
+$EndComp
+$Comp
+L power:GNDPWR #PWR?
+U 1 1 5F6435C9
+P 6650 3150
+F 0 "#PWR?" H 6650 2950 50  0001 C CNN
+F 1 "GNDPWR" H 6654 2996 50  0000 C CNN
+F 2 "" H 6650 3100 50  0001 C CNN
+F 3 "" H 6650 3100 50  0001 C CNN
+	1    6650 3150
+	1    0    0    -1
+$EndComp
+$Comp
+L power:+7.5V #PWR?
+U 1 1 5F6448FC
+P 6650 2650
+F 0 "#PWR?" H 6650 2500 50  0001 C CNN
+F 1 "+7.5V" H 6665 2823 50  0000 C CNN
+F 2 "" H 6650 2650 50  0001 C CNN
+F 3 "" H 6650 2650 50  0001 C CNN
+	1    6650 2650
+	1    0    0    -1
+$EndComp
+Wire Wire Line
+	6650 2650 6650 2750
+Wire Wire Line
+	6650 3050 6650 3150
 $EndSCHEMATC

Commit message: INI BOARD
Parts:
- added J1: Conn_01x05_NFC, Connector_JST:JST_GH_BM05B-GHS-TBT_1x05-1MP_P1.25mm_Vertical, symbol Connector_Generic:Conn_01x05
- added J2: Conn_01x03_Female_VibrationMotor, Connector_PinHeader_2.54mm:PinHeader_1x03_P2.54mm_Vertical, symbol Connector:Conn_01x03_Female
- gave numbers to parts that had none: 9
Connections:
- net +5V: now also A1.27 (+5V), J1.1 (Pin_1), J2.1 (Pin_1)
- net GND: now also A1.29 (GND), A1.4 (GND), J1.5 (Pin_5), J2.3 (Pin_3)
- net VibrationMotor: now reaches A1.1 (D1/TX)
- net VibrationMotor: now also J2.2 (Pin_2)
- net SCK: now reaches A1.16 (D13)
- net SCK: now also J1.2 (Pin_2)
- net SDA: now reaches A1.23 (A4)
- net SDA: now also J1.3 (Pin_3)
- net SCL: now reaches A1.24 (A5)
- net SCL: now also J1.4 (Pin_4)
Changed lines of the file:
@@
 $EndDescr
 $Comp
-L MCU_Module:Arduino_Nano_v2.x A?
+L MCU_Module:Arduino_Nano_v2.x A1
 U 1 1 5F46BD4B
 P 3750 3300
-F 0 "A?" H 3750 2211 50  0000 C CNN
+F 0 "A1" H 3750 2211 50  0000 C CNN
 F 1 "Arduino_Nano_v2.x" H 3750 2120 50  0000 C CNN
 F 2 "Module:Arduino_Nano_WithMountingHoles" H 3750 3300 50  0001 C CIN
@@
 $EndComp
 $Comp
-L LED:WS2812B D?
+L LED:WS2812B D1
 U 1 1 5F6043E7
 P 1100 1100
-F 0 "D?" H 1444 1146 50  0000 L CNN
+F 0 "D1" H 1444 1146 50  0000 L CNN
 F 1 "WS2812B" H 1444 1055 50  0000 L CNN
 F 2 "LED_SMD:LED_WS2812B_PLCC4_5.0x5.0mm_P3.2mm" H 1150 800 50  0001 L TNN
@@
 $EndComp
 $Comp
-L LED:WS2812B D?
+L LED:WS2812B D2
 U 1 1 5F606A1F
 P 2100 1100
-F 0 "D?" H 2444 1146 50  0000 L CNN
+F 0 "D2" H 2444 1146 50  0000 L CNN
 F 1 "WS2812B" H 2444 1055 50  0000 L CNN
 F 2 "LED_SMD:LED_WS2812B_PLCC4_5.0x5.0mm_P3.2mm" H 2150 800 50  0001 L TNN
@@
 $EndComp
 $Comp
-L LED:WS2812B D?
+L LED:WS2812B D3
 U 1 1 5F608368
 P 3100 1100
-F 0 "D?" H 3444 1146 50  0000 L CNN
+F 0 "D3" H 3444 1146 50  0000 L CNN
 F 1 "WS2812B" H 3444 1055 50  0000 L CNN
 F 2 "LED_SMD:LED_WS2812B_PLCC4_5.0x5.0mm_P3.2mm" H 3150 800 50  0001 L TNN
@@
 $EndComp
 $Comp
-L LED:WS2812B D?
+L LED:WS2812B D4
 U 1 1 5F60C729
 P 4100 1100
-F 0 "D?" H 4444 1146 50  0000 L CNN
+F 0 "D4" H 4444 1146 50  0000 L CNN
 F 1 "WS2812B" H 4444 1055 50  0000 L CNN
 F 2 "LED_SMD:LED_WS2812B_PLCC4_5.0x5.0mm_P3.2mm" H 4150 800 50  0001 L TNN
@@
 $EndComp
 $Comp
-L LED:WS2812B D?
+L LED:WS2812B D5
 U 1 1 5F60D2EA
 P 5100 1100
-F 0 "D?" H 5444 1146 50  0000 L CNN
+F 0 "D5" H 5444 1146 50  0000 L CNN
 F 1 "WS2812B" H 5444 1055 50  0000 L CNN
 F 2 "LED_SMD:LED_WS2812B_PLCC4_5.0x5.0mm_P3.2mm" H 5150 800 50  0001 L TNN
@@
 $EndComp
 $Comp
-L LED:WS2812B D?
+L LED:WS2812B D6
 U 1 1 5F60E008
 P 6100 1100
-F 0 "D?" H 6444 1146 50  0000 L CNN
+F 0 "D6" H 6444 1146 50  0000 L CNN
 F 1 "WS2812B" H 6444 1055 50  0000 L CNN
 F 2 "LED_SMD:LED_WS2812B_PLCC4_5.0x5.0mm_P3.2mm" H 6150 800 50  0001 L TNN
@@
 $EndComp
 $Comp
-L power:GND #PWR?
+L power:GND #PWR0101
 U 1 1 5F623C17
 P 6100 1500
-F 0 "#PWR?" H 6100 1250 50  0001 C CNN
+F 0 "#PWR0101" H 6100 1250 50  0001 C CNN
 F 1 "GND" H 6105 1327 50  0000 C CNN
 F 2 "" H 6100 1500 50  0001 C CNN
@@
 $EndComp
 $Comp
-L power:+5V #PWR?
+L power:+5V #PWR0102
 U 1 1 5F6244C7
 P 6100 700
-F 0 "#PWR?" H 6100 550 50  0001 C CNN
+F 0 "#PWR0102" H 6100 550 50  0001 C CNN
 F 1 "+5V" H 6115 873 50  0000 C CNN
 F 2 "" H 6100 700 50  0001 C CNN
@@
 NFC2
 $Comp
-L Mechanical:MountingHole_Pad H?
+L Mechanical:MountingHole_Pad H1
 U 1 1 5F64094E
 P 6800 1000
-F 0 "H?" H 6900 1049 50  0000 L CNN
+F 0 "H1" H 6900 1049 50  0000 L CNN
 F 1 "MountingHole_Pad" H 6900 958 50  0000 L CNN
 F 2 "Connector_PinHeader_1.00mm:PinHeader_1x01_P1.00mm_Vertical" H 6800 1000 50  0001 C CNN
@@
 $EndComp
 $Comp
-L Device:Battery_Cell BT?
+L Device:Battery_Cell BT1
 U 1 1 5F642495
 P 6650 2950
-F 0 "BT?" H 6768 3046 50  0000 L CNN
+F 0 "BT1" H 6768 3046 50  0000 L CNN
 F 1 "Battery_Cell" H 6768 2955 50  0000 L CNN
 F 2 "Connector_AMASS:AMASS_XT30U-F_1x02_P5.0mm_Vertical" V 6650 3010 50  0001 C CNN
@@
 $EndComp
 $Comp
-L power:GNDPWR #PWR?
+L power:GNDPWR #PWR0103
 U 1 1 5F6435C9
 P 6650 3150
-F 0 "#PWR?" H 6650 2950 50  0001 C CNN
+F 0 "#PWR0103" H 6650 2950 50  0001 C CNN
 F 1 "GNDPWR" H 6654 2996 50  0000 C CNN
 F 2 "" H 6650 3100 50  0001 C CNN
@@
 $EndComp
 $Comp
-L power:+7.5V #PWR?
+L power:+7.5V #PWR0104
 U 1 1 5F6448FC
 P 6650 2650
-F 0 "#PWR?" H 6650 2500 50  0001 C CNN
+F 0 "#PWR0104" H 6650 2500 50  0001 C CNN
 F 1 "+7.5V" H 6665 2823 50  0000 C CNN
 F 2 "" H 6650 2650 50  0001 C CNN
@@
 Wire Wire Line
 	6650 3050 6650 3150
+$Comp
+L Connector:Conn_01x03_Female J2
+U 1 1 5F60CF12
+P 5900 4000
+F 0 "J2" H 5928 4026 50  0000 L CNN
+F 1 "Conn_01x03_Female_VibrationMotor" H 5928 3935 50  0000 L CNN
+F 2 "Connector_PinHeader_2.54mm:PinHeader_1x03_P2.54mm_Vertical" H 5900 4000 50  0001 C CNN
+F 3 "~" H 5900 4000 50  0001 C CNN
+	1    5900 4000
+	1    0    0    -1
+$EndComp
+$Comp
+L power:+5V #PWR0105
+U 1 1 5F60E207
+P 5600 3850
+F 0 "#PWR0105" H 5600 3700 50  0001 C CNN
+F 1 "+5V" H 5615 4023 50  0000 C CNN
+F 2 "" H 5600 3850 50  0001 C CNN
+F 3 "" H 5600 3850 50  0001 C CNN
+	1    5600 3850
+	1    0    0    -1
+$EndComp
+$Comp
+L power:GND #PWR0106
+U 1 1 5F60F1E7
+P 5600 4150
+F 0 "#PWR0106" H 5600 3900 50  0001 C CNN
+F 1 "GND" H 5605 3977 50  0000 C CNN
+F 2 "" H 5600 4150 50  0001 C CNN
+F 3 "" H 5600 4150 50  0001 C CNN
+	1    5600 4150
+	1    0    0    -1
+$EndComp
+$Comp
+L power:GND #PWR0107
+U 1 1 5F60FD0B
+P 3850 4600
+F 0 "#PWR0107" H 3850 4350 50  0001 C CNN
+F 1 "GND" H 3855 4427 50  0000 C CNN
+F 2 "" H 3850 4600 50  0001 C CNN
+F 3 "" H 3850 4600 50  0001 C CNN
+	1    3850 4600
+	1    0    0    -1
+$EndComp
+$Comp
+L power:+5V #PWR0108
+U 1 1 5F611C0C
+P 3950 2200
+F 0 "#PWR0108" H 3950 2050 50  0001 C CNN
+F 1 "+5V" H 3965 2373 50  0000 C CNN
+F 2 "" H 3950 2200 50  0001 C CNN
+F 3 "" H 3950 2200 50  0001 C CNN
+	1    3950 2200
+	1    0    0    -1
+$EndComp
+Wire Wire Line
+	5700 3900 5600 3900
+Wire Wire Line
+	5600 3900 5600 3850
+Wire Wire Line
+	5700 4100 5600 4100
+Wire Wire Line
+	5600 4100 5600 4150
+Wire Wire Line
+	5700 4000 5150 4000
+Text Label 5150 4000 0    50   ~ 0
+VibrationMotor
+Wire Wire Line
+	3250 2800 2700 2800
+Text Label 2700 2800 0    50   ~ 0
+VibrationMotor
+Wire Wire Line
+	3250 4000 3050 4000
+Wire Wire Line
+	4250 3700 4450 3700
+Wire Wire Line
+	4250 3800 4450 3800
+Text Label 3050 4000 0    50   ~ 0
+SCK
+Text Label 4450 3700 2    50   ~ 0
+SDA
+Text Label 4450 3800 2    50   ~ 0
+SCL
+$Comp
+L Connector_Generic:Conn_01x05 J1
+U 1 1 5F618F19
+P 5850 4950
+F 0 "J1" H 5930 4992 50  0000 L CNN
+F 1 "Conn_01x05_NFC" H 5930 4901 50  0000 L CNN
+F 2 "Connector_JST:JST_GH_BM05B-GHS-TBT_1x05-1MP_P1.25mm_Vertical" H 5850 4950 50  0001 C CNN
+F 3 "~" H 5850 4950 50  0001 C CNN
+	1    5850 4950
+	1    0    0    -1
+$EndComp
+Wire Wire Line
+	3850 4600 3850 4350
+Wire Wire Line
+	3750 4300 3750 4350
+Wire Wire Line
+	3750 4350 3850 4350
+Connection ~ 3850 4350
+Wire Wire Line
+	3850 4350 3850 4300
+Wire Wire Line
+	3950 2300 3950 2200
+$Comp
+L power:+5V #PWR0109
+U 1 1 5F61CB4E
+P 5550 4650
+F 0 "#PWR0109" H 5550 4500 50  0001 C CNN
+F 1 "+5V" H 5565 4823 50  0000 C CNN
+F 2 "" H 5550 4650 50  0001 C CNN
+F 3 "" H 5550 4650 50  0001 C CNN
+	1    5550 4650
+	1    0    0    -1
+$EndComp
+$Comp
+L power:GND #PWR0110
+U 1 1 5F61DE76
+P 5550 5250
+F 0 "#PWR0110" H 5550 5000 50  0001 C CNN
+F 1 "GND" H 5555 5077 50  0000 C CNN
+F 2 "" H 5550 5250 50  0001 C CNN
+F 3 "" H 5550 5250 50  0001 C CNN
+	1    5550 5250
+	1    0    0    -1
+$EndComp
+Wire Wire Line
+	5650 5150 5550 5150
+Wire Wire Line
+	5550 5150 5550 5250
+Wire Wire Line
+	5550 4650 5550 4750
+Wire Wire Line
+	5550 4750 5650 4750
+Wire Wire Line
+	5650 4850 5400 4850
+Wire Wire Line
+	5650 4950 5400 4950
+Wire Wire Line
+	5650 5050 5400 5050
+Text Label 5400 4850 0    50   ~ 0
+SCK
+Text Label 5400 4950 0    50   ~ 0
+SDA
+Text Label 5400 5050 0    50   ~ 0
+SCL
 $EndSCHEMATC

Commit message: finish PCB
Connections:
- net +7.5V is gone; now on net +5V: BT1.1 (+)
- net GNDPWR is gone; now on net GND: BT1.2 (-)
Other:
- moved on the sheet: A1, BT1, J1, J2

Commit message: NFC ini
Parts:
- removed H1: MountingHole_Pad, Connector_PinHeader_1.00mm:PinHeader_1x01_P1.00mm_Vertical, symbol Mechanical:MountingHole_Pad
- removed J1: Conn_01x05_NFC, Connector_JST:JST_GH_BM05B-GHS-TBT_1x05-1MP_P1.25mm_Vertical, symbol Connector_Generic:Conn_01x05
- added J1: Conn_01x04_NFC, Connector_JST:JST_GH_BM04B-GHS-TBT_1x04-1MP_P1.25mm_Vertical, symbol Connector_Generic:Conn_01x04
- BT1: footprint Connector_AMASS:AMASS_XT30U-F_1x02_P5.0mm_Vertical -> Connector_JST:JST_PH_B2B-PH-K_1x02_P2.00mm_Vertical
Connections:
- net +5V: now also J1.1 (Pin_1)
- net GND: now also J1.4 (Pin_4)
- net SCL: now also J1.3 (Pin_3)
- net SDA: now also J1.2 (Pin_2)
- net VibrationMotor: now also A1.5 (D2); no longer A1.1 (D1/TX)
- net SCK: no longer names the net of A1.16 (D13)
Other:
- moved on the sheet: A1, BT1, D1, D2, D3, D4, D5, D6, J2
