File: KiCAD/NFC/NFC.sch (KiCad schematic (older format))
At the start: 1 part

Commit message: NFC coil
Parts:
- added J2: Conn_01x03_EnergyHarvesting, Connector_JST:JST_GH_BM03B-GHS-TBT_1x03-1MP_P1.25mm_Vertical, symbol Connector_Generic:Conn_01x03
- added L1: NFC, NFC:Class6NFC, symbol Device:L
- added U1: NTA53321G0FFT, Package_SO:TSSOP-16_4.4x5mm_P0.65mm, symbol NFC:NTA53321G0FFT
- J1: renamed from J?; value Conn_01x04 -> Conn_01x04_I2C
Connections:
- net +5V: now also U1.11 (VCC)
- net GND: now also J2.3 (Pin_3), U1.13 (GND), U1.3 (GND), U1.4 (GNDTX)
- net SCL: now also U1.9 (SCL/GPIO0/PWM0)
- net SDA: now also U1.8 (SDA/GPIO1/PWM1)
- new net ED: J2.2 (Pin_2), U1.10 (ED/PWM0)
- new net LA: L1.1, U1.1 (LA)
- new net LB: L1.2, U1.16 (LB)
- new net VOUT: J2.1 (Pin_1), U1.14 (VOUT)
Other:
- moved on the sheet: J1
Changed lines of the file:
@@
 $EndDescr
 $Comp
-L Connector_Generic:Conn_01x04 J?
+L Connector_Generic:Conn_01x04 J1
 U 1 1 5F61EBF3
-P 3000 1850
-F 0 "J?" H 3080 1842 50  0000 L CNN
-F 1 "Conn_01x04" H 3080 1751 50  0000 L CNN
-F 2 "Connector_JST:JST_GH_BM04B-GHS-TBT_1x04-1MP_P1.25mm_Vertical" H 3000 1850 50  0001 C CNN
-F 3 "~" H 3000 1850 50  0001 C CNN
-	1    3000 1850
-	1    0    0    -1
-$EndComp
-Wire Wire Line
-	2800 1850 2550 1850
-Wire Wire Line
-	2800 1950 2550 1950
-$Comp
-L power:+5V #PWR?
+P 3000 1700
+F 0 "J1" H 3080 1692 50  0000 L CNN
+F 1 "Conn_01x04_I2C" H 3080 1601 50  0000 L CNN
+F 2 "Connector_JST:JST_GH_BM04B-GHS-TBT_1x04-1MP_P1.25mm_Vertical" H 3000 1700 50  0001 C CNN
+F 3 "~" H 3000 1700 50  0001 C CNN
+	1    3000 1700
+	1    0    0    -1
+$EndComp
+Wire Wire Line
+	2800 1700 2550 1700
+Wire Wire Line
+	2800 1800 2550 1800
+$Comp
+L power:+5V #PWR0101
 U 1 1 5F621D21
-P 2700 1650
-F 0 "#PWR?" H 2700 1500 50  0001 C CNN
-F 1 "+5V" H 2715 1823 50  0000 C CNN
-F 2 "" H 2700 1650 50  0001 C CNN
-F 3 "" H 2700 1650 50  0001 C CNN
-	1    2700 1650
-	1    0    0    -1
-$EndComp
-$Comp
-L power:GND #PWR?
+P 2700 1500
+F 0 "#PWR0101" H 2700 1350 50  0001 C CNN
+F 1 "+5V" H 2715 1673 50  0000 C CNN
+F 2 "" H 2700 1500 50  0001 C CNN
+F 3 "" H 2700 1500 50  0001 C CNN
+	1    2700 1500
+	1    0    0    -1
+$EndComp
+$Comp
+L power:GND #PWR0102
 U 1 1 5F6230CA
-P 2700 2150
-F 0 "#PWR?" H 2700 1900 50  0001 C CNN
-F 1 "GND" H 2705 1977 50  0000 C CNN
-F 2 "" H 2700 2150 50  0001 C CNN
-F 3 "" H 2700 2150 50  0001 C CNN
-	1    2700 2150
-	1    0    0    -1
-$EndComp
-Wire Wire Line
-	2800 2050 2700 2050
-Wire Wire Line
-	2700 2050 2700 2150
-Wire Wire Line
-	2800 1750 2700 1750
-Wire Wire Line
-	2700 1750 2700 1650
-Text Label 2550 1850 0    50   ~ 0
+P 2700 2000
+F 0 "#PWR0102" H 2700 1750 50  0001 C CNN
+F 1 "GND" H 2705 1827 50  0000 C CNN
+F 2 "" H 2700 2000 50  0001 C CNN
+F 3 "" H 2700 2000 50  0001 C CNN
+	1    2700 2000
+	1    0    0    -1
+$EndComp
+Wire Wire Line
+	2800 1900 2700 1900
+Wire Wire Line
+	2700 1900 2700 2000
+Wire Wire Line
+	2800 1600 2700 1600
+Wire Wire Line
+	2700 1600 2700 1500
+Text Label 2550 1700 0    50   ~ 0
 SDA
-Text Label 2550 1950 0    50   ~ 0
+Text Label 2550 1800 0    50   ~ 0
 SCL
+$Comp
+L NFC:NTA53321G0FFT U1
+U 1 1 5F63D709
+P 3800 3550
+F 0 "U1" H 3800 4615 50  0000 C CNN
+F 1 "NTA53321G0FFT" H 3800 4524 50  0000 C CNN
+F 2 "Package_SO:TSSOP-16_4.4x5mm_P0.65mm" H 3800 3250 50  0001 C CNN
+F 3 "https://www.nxp.com.cn/part/NTA53321G0FTT#/" H 3800 3550 50  0001 C CNN
+	1    3800 3550
+	1    0    0    -1
+$EndComp
+$Comp
+L Device:L L1
+U 1 1 5F642323
+P 3750 3950
+F 0 "L1" V 3940 3950 50  0000 C CNN
+F 1 "NFC" V 3849 3950 50  0000 C CNN
+F 2 "NFC:Class6NFC" H 3750 3950 50  0001 C CNN
+F 3 "~" H 3750 3950 50  0001 C CNN
+	1    3750 3950
+	0    -1   -1   0
+$EndComp
+$Comp
+L power:GND #PWR0103
+U 1 1 5F645F01
+P 5050 3550
+F 0 "#PWR0103" H 5050 3300 50  0001 C CNN
+F 1 "GND" H 5055 3377 50  0000 C CNN
+F 2 "" H 5050 3550 50  0001 C CNN
+F 3 "" H 5050 3550 50  0001 C CNN
+	1    5050 3550
+	1    0    0    -1
+$EndComp
+$Comp
+L power:GND #PWR0104
+U 1 1 5F6486EE
+P 2550 3550
+F 0 "#PWR0104" H 2550 3300 50  0001 C CNN
+F 1 "GND" H 2555 3377 50  0000 C CNN
+F 2 "" H 2550 3550 50  0001 C CNN
+F 3 "" H 2550 3550 50  0001 C CNN
+	1    2550 3550
+	1    0    0    -1
+$EndComp
+Wire Wire Line
+	4700 3450 4950 3450
+Wire Wire Line
+	2900 3450 2650 3450
+Text Label 4950 3450 2    50   ~ 0
+SCL
+Text Label 2650 3450 0    50   ~ 0
+SDA
+Wire Wire Line
+	4700 2750 4950 2750
+Wire Wire Line
+	2900 2750 2650 2750
+Text Label 2650 2750 0    50   ~ 0
+LA
+Text Label 4950 2750 2    50   ~ 0
+LB
+Wire Wire Line
+	5050 3550 5050 3050
+Wire Wire Line
+	5050 3050 4700 3050
+Wire Wire Line
+	2550 3550 2550 2950
+Wire Wire Line
+	2550 2950 2650 2950
+Wire Wire Line
+	2900 3050 2650 3050
+Wire Wire Line
+	2650 3050 2650 2950
+Connection ~ 2650 2950
+Wire Wire Line
+	2650 2950 2900 2950
+$Comp
+L Graphic:SYM_ESD_Large #SYM1
+U 1 1 5F651CEE
+P 3150 4400
+F 0 "#SYM1" H 3150 4600 50  0001 C CNN
+F 1 "SYM_ESD_Large" H 3150 4150 50  0001 C CNN
+F 2 "Symbol:ESD-Logo_22x20mm_SilkScreen" H 3145 4370 50  0001 C CNN
+F 3 "~" H 3145 4370 50  0001 C CNN
+	1    3150 4400
+	1    0    0    -1
+$EndComp
+$Comp
+L Graphic:Logo_Open_Hardware_Small #LOGO1
+U 1 1 5F654FA5
+P 4400 4450
+F 0 "#LOGO1" H 4400 4725 50  0001 C CNN
+F 1 "Logo_Open_Hardware_Small" H 4400 4225 50  0001 C CNN
+F 2 "Symbol:KiCad-Logo2_6mm_SilkScreen" H 4400 4450 50  0001 C CNN
+F 3 "~" H 4400 4450 50  0001 C CNN
+	1    4400 4450
+	1    0    0    -1
+$EndComp
+Wire Wire Line
+	4700 3350 4950 3350
+Text Label 4950 3350 2    50   ~ 0
+ED
+$Comp
+L Connector_Generic:Conn_01x03 J2
+U 1 1 5F6566DE
+P 4350 1750
+F 0 "J2" H 4430 1792 50  0000 L CNN
+F 1 "Conn_01x03_EnergyHarvesting" H 4430 1701 50  0000 L CNN
+F 2 "Connector_JST:JST_GH_BM03B-GHS-TBT_1x03-1MP_P1.25mm_Vertical" H 4350 1750 50  0001 C CNN
+F 3 "~" H 4350 1750 50  0001 C CNN
+	1    4350 1750
+	1    0    0    -1
+$EndComp
+Wire Wire Line
+	4150 1750 3900 1750
+Wire Wire Line
+	4150 1650 3900 1650
+Wire Wire Line
+	4700 2950 4950 2950
+Text Label 4950 2950 2    50   ~ 0
+VOUT
+Text Label 3900 1650 0    50   ~ 0
+VOUT
+Text Label 3900 1750 0    50   ~ 0
+ED
+$Comp
+L power:GND #PWR0105
+U 1 1 5F6596A7
+P 3900 1950
+F 0 "#PWR0105" H 3900 1700 50  0001 C CNN
+F 1 "GND" H 3905 1777 50  0000 C CNN
+F 2 "" H 3900 1950 50  0001 C CNN
+F 3 "" H 3900 1950 50  0001 C CNN
+	1    3900 1950
+	1    0    0    -1
+$EndComp
+Wire Wire Line
+	3900 1850 3900 1950
+Wire Wire Line
+	3900 1850 4150 1850
+Wire Wire Line
+	3600 3950 3350 3950
+Wire Wire Line
+	3900 3950 4150 3950
+Text Label 4150 3950 2    50   ~ 0
+LB
+Text Label 3350 3950 0    50   ~ 0
+LA
+$Comp
+L power:+5V #PWR0106
+U 1 1 5F670AC3
+P 4800 3250
+F 0 "#PWR0106" H 4800 3100 50  0001 C CNN
+F 1 "+5V" V 4815 3378 50  0000 L CNN
+F 2 "" H 4800 3250 50  0001 C CNN
+F 3 "" H 4800 3250 50  0001 C CNN
+	1    4800 3250
+	0    1    1    0
+$EndComp
+Wire Wire Line
+	4700 3250 4800 3250
 $EndSCHEMATC
